File: pcb.kicad_pcb (KiCad board)
At the start: 2 copper layers, 100 x 100 mm, 26 parts, among them J1 Screw_Terminal_01x04, J2 USB_C_Receptacle_PowerOnly_6P, J3 Screw_Terminal_01x04, J5 USB_B_Micro, J6 DC5.5x2.1, J7 DC5.5x2.1

Commit message: ready to production
Parts:
- added C1: 0.1uf, Capacitor_SMD:C_0603_1608Metric_Pad1.08x0.95mm_HandSolder, F.Cu at (154.8, 126.2)
- added C2: 0.1uf, Capacitor_SMD:C_0603_1608Metric_Pad1.08x0.95mm_HandSolder, F.Cu at (157.3, 126.2)
- added C3: 10uf, Capacitor_THT:CP_Radial_D5.0mm_P2.50mm, F.Cu at (164.9, 125.3)
- added C4: 10uf, Capacitor_THT:CP_Radial_D5.0mm_P2.50mm, F.Cu at (164.9, 138.0)
- added D1: LED, LED_THT:LED_D4.0mm, F.Cu at (169.9, 131.2)
- added J1: Conn_01x05_Socket, libs:pads_01x05_P2.00mm_Vertical_SMD, F.Cu at (98.3, 135.5)
- added J2: Conn_02x05_Odd_Even, Connector_PinHeader_2.00mm:PinHeader_2x05_P2.00mm_Vertical, F.Cu at (118.9, 130.1)
- added J4: Conn_02x04_Counter_Clockwise, libs:PS2x04_P2.54mm_Vertical_sequential, F.Cu at (192.8, 125.3)
- added J5: Conn_01x05_Socket, libs:pads_01x05_P2.00mm_Vertical_SMD, B.Cu at (103.4, 135.5)
- added J6: Conn_02x05_Odd_Even, Connector_PinHeader_2.54mm:PinHeader_2x05_P2.54mm_Vertical, F.Cu at (123.2, 136.7)
- added J7: USB_B_Micro, libs:USB_Micro-B_Amphenol_10103594-0001LF_Horizontal, F.Cu at (180.4, 121.9)
- added JP10: Jumper_3_Open, Connector_PinHeader_2.54mm:PinHeader_1x03_P2.54mm_Vertical, F.Cu at (188.8, 143.9)
- added JP3: Jumper_3_Open, libs:jumper3_1x04_P2.54mm_Vertical, F.Cu at (132.8, 124.6)
- added JP4: Jumper_3_Open, libs:jumper3_1x04_P2.54mm_Vertical, F.Cu at (139.5, 124.6)
- added JP5: Jumper_3_Open, libs:jumper3_1x04_P2.54mm_Vertical, F.Cu at (146.2, 124.6)
- added JP6: Jumper_3_Open, libs:jumper3_1x04_P2.54mm_Vertical, F.Cu at (132.4, 138.6)
- added JP7: Jumper_3_Open, libs:jumper3_1x04_P2.54mm_Vertical, F.Cu at (139.1, 138.6)
- added JP8: Jumper_3_Open, libs:jumper3_1x04_P2.54mm_Vertical, F.Cu at (145.9, 138.6)
- added JP9: Jumper_3_Open, Connector_PinHeader_2.54mm:PinHeader_1x03_P2.54mm_Vertical, F.Cu at (177.6, 130.4)
- added R17: 1k, Resistor_SMD:R_0603_1608Metric_Pad0.98x0.95mm_HandSolder, F.Cu at (154.7, 144.0)
- added R18: 1k, Resistor_SMD:R_0603_1608Metric_Pad0.98x0.95mm_HandSolder, F.Cu at (157.3, 144.0)
- added R19: 1k, Resistor_SMD:R_0603_1608Metric_Pad0.98x0.95mm_HandSolder, F.Cu at (162.4, 144.0)
- added R20: 1k, Resistor_SMD:R_0603_1608Metric_Pad0.98x0.95mm_HandSolder, F.Cu at (164.9, 144.0)
- added R21: 1k, Resistor_SMD:R_0603_1608Metric_Pad0.98x0.95mm_HandSolder, F.Cu at (170.0, 144.0)
- added R3: 270, Resistor_SMD:R_0805_2012Metric_Pad1.20x1.40mm_HandSolder, F.Cu at (172.2, 121.2)
- added U1: TXB0104E, Package_SO:TSSOP-14_4.4x5mm_P0.65mm, F.Cu at (157.3, 132.9)
- added U2: AMS1117-1.8, Package_TO_SOT_SMD:SOT-223-3_TabPin2, F.Cu at (176.6, 138.3)
- added U4: AMS1117-3.3, Package_TO_SOT_SMD:SOT-223-3_TabPin2, B.Cu at (179.6, 138.3)
Routing:
- net (no net): track 1284.9 -> 2785.1 mm, vias 0 -> 37
Other:
- board size 100 x 100 mm -> 100 x 96.5 mm
- board text added: "+"
- board text added: "J1/J2/J6 to MB"
- board text added: "JP10:12=ext_usb_pwr,23=programmer JP9:12=1.8v,23=3.3v"
- board text added: "MB Jumpers: 12=ASUS 23=ASROCK 24=MSI"
- board text added: "pullup R17-R20 if use TXB010x instead of TXS010x."
